Commit message: Simulation Environment

File: amr_manipulator_description/urdf/amr_manipulator.urdf.xacro (robot description, xacro)
@@ -7,5 +7,12 @@
   <xacro:include filename="$(find amr_manipulator_description)/urdf/sensors/rgbd_camera.urdf.xacro"/>
   <xacro:property name="ur_cfg" value="$(find amr_manipulator_description)/config/arm/ur5e"/>
+  <xacro:arg name="use_sim" default="false"/>
   <xacro:mobile_base/>
+  <!-- UR5e joint dynamics, used by the Gazebo physics (damping in N*m*s/rad, friction in N*m).
+       Round numbers chosen so the arm settles in a few seconds: NOT identified on a real UR5e. -->
+  <xacro:property name="ur_damping_large" value="2.0"/>
+  <xacro:property name="ur_damping_wrist" value="0.5"/>
+  <xacro:property name="ur_friction_large" value="1.0"/>
+  <xacro:property name="ur_friction_wrist" value="0.3"/>
   <xacro:ur_robot
     name="ur5e"
@@ -17,5 +24,9 @@
     visual_parameters_file="${ur_cfg}/visual_parameters.yaml"
     ur_type="ur5e"
-    generate_ros2_control_tag="false">
+    generate_ros2_control_tag="false"
+    joint_damping_large="${ur_damping_large}"
+    joint_damping_wrist="${ur_damping_wrist}"
+    joint_friction_large="${ur_friction_large}"
+    joint_friction_wrist="${ur_friction_wrist}">
     <origin xyz="0 0 0" rpy="0 0 0"/>
   </xacro:ur_robot>
@@ -29,3 +40,8 @@
     <origin xyz="0.0425 0 0.03" rpy="0 ${-pi/2} 0"/>
   </xacro:rgbd_camera>
+  <xacro:if value="$(arg use_sim)">
+    <xacro:include filename="$(find amr_manipulator_description)/urdf/sim/gazebo_physics.xacro"/>
+    <xacro:include filename="$(find amr_manipulator_description)/urdf/sim/gazebo_plugins.xacro"/>
+    <xacro:include filename="$(find amr_manipulator_description)/urdf/sim/ros2_control.xacro"/>
+  </xacro:if>
 </robot>

File: amr_manipulator_description/urdf/arm/ur_macro.xacro (robot description, xacro)
@@ -44,4 +44,12 @@
   <xacro:include filename="$(find amr_manipulator_description)/urdf/arm/inc/ur_transmissions.xacro" />
   <xacro:include filename="$(find amr_manipulator_description)/urdf/arm/inc/ur_common.xacro" />
+  <!--
+    MODIFIED for amr_manipulator (original: UniversalRobots/Universal_Robots_ROS2_Description, humble):
+    - the include paths point to this package;
+    - new parameters joint_damping_large / joint_damping_wrist / joint_friction_large /
+      joint_friction_wrist set the <dynamics> of the joints used by the Gazebo physics
+      (large = shoulder_pan, shoulder_lift, elbow; wrist = wrist_1, wrist_2, wrist_3).
+      Default 0.0 = upstream behaviour. Damping in N*m*s/rad, friction in N*m.
+  -->
   <xacro:macro name="ur_robot" params="
     name
@@ -63,4 +71,8 @@
     sim_gazebo:=false
     sim_ignition:=false
+    joint_damping_large:=0.0
+    joint_damping_wrist:=0.0
+    joint_friction_large:=0.0
+    joint_friction_wrist:=0.0
     headless_mode:=false
     initial_positions:=${dict(shoulder_pan_joint=0.0,shoulder_lift_joint=-1.57,elbow_joint=0.0,wrist_1_joint=-1.57,wrist_2_joint=0.0,wrist_3_joint=0.0)}
@@ -352,5 +364,5 @@
          <safety_controller soft_lower_limit="${shoulder_pan_lower_limit + safety_pos_margin}" soft_upper_limit="${shoulder_pan_upper_limit - safety_pos_margin}" k_position="${safety_k_position}" k_velocity="0.0"/>
       </xacro:if>
-      <dynamics damping="0" friction="0"/>
+      <dynamics damping="${joint_damping_large}" friction="${joint_friction_large}"/>
     </joint>
     <joint name="${tf_prefix}shoulder_lift_joint" type="revolute">
@@ -364,5 +376,5 @@
          <safety_controller soft_lower_limit="${shoulder_lift_lower_limit + safety_pos_margin}" soft_upper_limit="${shoulder_lift_upper_limit - safety_pos_margin}" k_position="${safety_k_position}" k_velocity="0.0"/>
       </xacro:if>
-      <dynamics damping="0" friction="0"/>
+      <dynamics damping="${joint_damping_large}" friction="${joint_friction_large}"/>
     </joint>
     <joint name="${tf_prefix}elbow_joint" type="revolute">
@@ -376,5 +388,5 @@
          <safety_controller soft_lower_limit="${elbow_joint_lower_limit + safety_pos_margin}" soft_upper_limit="${elbow_joint_upper_limit - safety_pos_margin}" k_position="${safety_k_position}" k_velocity="0.0"/>
       </xacro:if>
-      <dynamics damping="0" friction="0"/>
+      <dynamics damping="${joint_damping_large}" friction="${joint_friction_large}"/>
     </joint>
     <joint name="${tf_prefix}wrist_1_joint" type="revolute">
@@ -388,5 +400,5 @@
          <safety_controller soft_lower_limit="${wrist_1_lower_limit + safety_pos_margin}" soft_upper_limit="${wrist_1_upper_limit - safety_pos_margin}" k_position="${safety_k_position}" k_velocity="0.0"/>
       </xacro:if>
-      <dynamics damping="0" friction="0"/>
+      <dynamics damping="${joint_damping_wrist}" friction="${joint_friction_wrist}"/>
     </joint>
     <joint name="${tf_prefix}wrist_2_joint" type="revolute">
@@ -400,5 +412,5 @@
          <safety_controller soft_lower_limit="${wrist_2_lower_limit + safety_pos_margin}" soft_upper_limit="${wrist_2_upper_limit - safety_pos_margin}" k_position="${safety_k_position}" k_velocity="0.0"/>
       </xacro:if>
-      <dynamics damping="0" friction="0"/>
+      <dynamics damping="${joint_damping_wrist}" friction="${joint_friction_wrist}"/>
     </joint>
     <joint name="${tf_prefix}wrist_3_joint" type="${wrist_3_joint_type}">
@@ -420,5 +432,5 @@
         </xacro:if>
       </xacro:unless>
-      <dynamics damping="0" friction="0"/>
+      <dynamics damping="${joint_damping_wrist}" friction="${joint_friction_wrist}"/>
     </joint>
     <link name="${tf_prefix}ft_frame"/>
